Commit message: fix : urdf file

File: esibot_description/urdf/esibot.urdf.xacro (robot description, xacro)
@@ -16,5 +16,5 @@
         │   │       └── ultrasound_sensor (fixed, HC-SR04 board)
         │   └── camera_link (fixed, ESP32-CAM)
-        │       └── camera_optical_link (fixed, Z-forward optical frame)
+        │       └── camera_optical_frame (fixed, Z-forward optical frame)
         └── imu_link (fixed, placeholder)
   Materials / Gazebo surface props → materials.xacro  (do NOT redeclare here)
@@ -208,5 +208,5 @@
     </inertial>
   </link>
-  <link name="camera_optical_link"/>
+  <link name="camera_optical_frame"/>
   <joint name="camera_joint" type="fixed">
     <parent link="upper_plate"/>
@@ -216,5 +216,5 @@
   <joint name="camera_optical_joint" type="fixed">
     <parent link="camera_link"/>
-    <child  link="camera_optical_link"/>
+    <child  link="camera_optical_frame"/>
     <origin xyz="0 0 0" rpy="${-pi/2} 0 ${-pi/2}"/>
   </joint>

Commit message: chore : fix urdf

File: esibot_description/urdf/esibot.urdf.xacro (robot description, xacro)
@@ -3,20 +3,20 @@
   EsiBot URDF/Xacro
   ==================
-  Architecture : 2-wheel differential drive + 1 caster + SG90 servo turret + HC-SR04 + ESP32-CAM
-  Matches spec : HC-SR04 on SG90 servo = pseudo-LiDAR  |  ESP32-CAM OV2640 camera
-  TF tree:
-    base_footprint  (Nav2/SLAM root, ground level)
-    └── base_link   (lower chassis centre)
-        ├── left_wheel   (continuous)
-        ├── right_wheel  (continuous)
-        ├── caster_wheel (fixed)
-        ├── upper_plate  (fixed, 80 mm above)
-        │   ├── servo_base  (fixed, SG90 body)
-        │   │   └── servo_link  (REVOLUTE ±90°, drives HC-SR04 sweep)
-        │   │       └── ultrasound_sensor (fixed, HC-SR04 board)
-        │   └── camera_link (fixed, ESP32-CAM)
-        │       └── camera_optical_frame (fixed, Z-forward optical frame)
-        └── imu_link (fixed, placeholder)
-  Materials / Gazebo surface props → materials.xacro  (do NOT redeclare here)
+  ── TF tree ────────────────────────────────────────────────────────────────
+  map (provided at runtime by SLAM / AMCL — NOT in URDF)
+  └── odom (provided at runtime by diff-drive odometry node — NOT in URDF)
+      └── base_footprint  (Nav2/SLAM root, ground level)
+          └── base_link   (lower chassis centre)
+              ├── left_wheel   (continuous)
+              ├── right_wheel  (continuous)
+              ├── caster_wheel (fixed)
+              ├── imu_link     (fixed, placeholder)
+              └── upper_plate  (fixed, 80 mm above base_link)
+                  ├── servo_base  (fixed — SG90 body)
+                  │   └── servo_link  (REVOLUTE ±90°, sweeps HC-SR04)
+                  │       └── laser_link  (fixed — HC-SR04 board, published as LaserScan frame)
+                  └── camera_link (fixed — ESP32-CAM board)
+                      └── camera_optical_frame (fixed — Z-forward ROS optical convention)
+  ───────────────────────────────────────────────────────────────────────────
 -->
 <robot name="esibot" xmlns:xacro="http://www.ros.org/wiki/xacro">
@@ -32,5 +32,5 @@
   <xacro:property name="caster_radius"    value="0.010"/>
   <xacro:property name="spacer_height"    value="0.080"/>
-  <xacro:property name="sensor_arm_x"     value="0.020"/>
+  <xacro:property name="sensor_arm_x"    value="0.020"/>
   <!-- ── BASE FOOTPRINT ───────────────────────────────────────────────────── -->
   <link name="base_footprint"/>
@@ -144,11 +144,4 @@
   </joint>
   <!-- ── SERVO LINK (SG90 horn — REVOLUTE) ────────────────────────────────── -->
-  <!--
-    angle =   0   → sensor faces forward (+X)
-    angle = +π/2  → sensor faces left    (+Y)
-    angle = -π/2  → sensor faces right   (-Y)
-    The Gazebo joint_state_publisher plugin publishes this angle to /joint_states.
-    NEVER run joint_state_publisher_gui alongside Gazebo — they conflict.
-  -->
   <link name="servo_link">
     <visual>
@@ -170,9 +163,9 @@
     <origin xyz="0 0 0.016" rpy="0 0 0"/>
     <axis xyz="0 0 1"/>
-    <limit lower="${-pi/2}" upper="${pi/2}" effort="0.34" velocity="5.24"/>
+    <limit lower="0.0" upper="${pi}" effort="0.34" velocity="5.24"/>
     <dynamics damping="0.001" friction="0.001"/>
   </joint>
-  <!-- ── HC-SR04 SENSOR LINK ──────────────────────────────────────────────── -->
-  <link name="ultrasound_sensor">
+  <!-- ── LASER LINK (HC-SR04 ultrasonic sensor board) ─────────────────────── -->
+  <link name="laser_link">
     <visual>
       <geometry><box size="0.045 0.020 0.015"/></geometry>
@@ -188,7 +181,7 @@
     </inertial>
   </link>
-  <joint name="ultrasound_joint" type="fixed">
+  <joint name="laser_joint" type="fixed">
     <parent link="servo_link"/>
-    <child  link="ultrasound_sensor"/>
+    <child  link="laser_link"/>
     <origin xyz="${sensor_arm_x} 0 0.010" rpy="0 0 0"/>
   </joint>
@@ -257,5 +250,5 @@
 </gazebo>
 <!-- 3. HC-SR04 Ray Sensor -->
-<gazebo reference="ultrasound_sensor">
+<gazebo reference="laser_link">
   <sensor name="ultrasound" type="gpu_lidar">
     <always_on>true</always_on>

File: esibot_description/urdf/materials.xacro (robot description, xacro)
@@ -125,5 +125,5 @@
   </gazebo>
   <!-- HC-SR04 sensor -->
-  <gazebo reference="ultrasound_sensor">
+  <gazebo reference="laser_link">
     <material>Gazebo/Blue</material>
   </gazebo>

Commit message: chore:fix /scan topic

File: esibot_description/urdf/esibot.urdf.xacro (robot description, xacro)
@@ -163,5 +163,5 @@
     <origin xyz="0 0 0.016" rpy="0 0 0"/>
     <axis xyz="0 0 1"/>
-    <limit lower="0.0" upper="${pi}" effort="0.34" velocity="5.24"/>
+    <limit lower="${-pi/2}" upper="${pi/2}" effort="0.34" velocity="5.24"/>
     <dynamics damping="0.001" friction="0.001"/>
   </joint>

Commit message: fix(sensors,urdf,slam): radar_node rewrite with thread sweep, extend servo joint limits to ±π, lower slam min travel thresholds

File: esibot_description/urdf/esibot.urdf.xacro (robot description, xacro)
@@ -163,5 +163,5 @@
     <origin xyz="0 0 0.016" rpy="0 0 0"/>
     <axis xyz="0 0 1"/>
-    <limit lower="${-pi/2}" upper="${pi/2}" effort="0.34" velocity="5.24"/>
+    <limit lower="${-pi}" upper="${pi}" effort="0.34" velocity="5.24"/>
     <dynamics damping="0.001" friction="0.001"/>
   </joint>

Commit message: dashboard status badges + fix incosistency + nav2 launching

File: esibot_description/urdf/esibot.urdf.xacro (robot description, xacro)
@@ -24,10 +24,10 @@
   <xacro:include filename="$(find esibot_description)/urdf/materials.xacro"/>
   <!-- ── Properties — update with real chassis measurements ────────────────── -->
-  <xacro:property name="base_width"       value="0.138"/>
+  <xacro:property name="base_width"       value="0.160"/>
   <xacro:property name="base_length"      value="0.140"/>
   <xacro:property name="base_height"      value="0.012"/>
   <xacro:property name="wheel_radius"     value="0.033"/>
   <xacro:property name="wheel_width"      value="0.018"/>
-  <xacro:property name="wheel_separation" value="0.138"/>
+  <xacro:property name="wheel_separation" value="0.160"/>
   <xacro:property name="caster_radius"    value="0.010"/>
   <xacro:property name="spacer_height"    value="0.080"/>
