Commit message: fix(nav2,urdf,ui): tune nav2 for Pi 4 perf, revert URDF to original values
- nav2_params: controller_frequency 5→1 Hz, costmap updates 0.5→0.2 Hz,
  movement_time_allowance 10→30s, bond_timeout 30s for Pi 4
- full.launch.py: nav2 start delay 15→25s for AMCL map→odom TF convergence
- urdf: revert base_width/wheel_separation to 0.138 (user-confirmed values)
- useServo: fix topic name /esibot/servo_angle → /servo_angle
- esibot_ui: rebuild bundle

Co-Authored-By: Claude Opus 4.6 <noreply@anthropic.com>

File: esibot_description/urdf/esibot.urdf.xacro (robot description, xacro)
@@ -24,10 +24,10 @@
   <xacro:include filename="$(find esibot_description)/urdf/materials.xacro"/>
   <!-- ── Properties — update with real chassis measurements ────────────────── -->
-  <xacro:property name="base_width"       value="0.160"/>
+  <xacro:property name="base_width"       value="0.138"/>
   <xacro:property name="base_length"      value="0.140"/>
   <xacro:property name="base_height"      value="0.012"/>
   <xacro:property name="wheel_radius"     value="0.033"/>
   <xacro:property name="wheel_width"      value="0.018"/>
-  <xacro:property name="wheel_separation" value="0.160"/>
+  <xacro:property name="wheel_separation" value="0.138"/>
   <xacro:property name="caster_radius"    value="0.010"/>
   <xacro:property name="spacer_height"    value="0.080"/>
